File: _restore_backup_2026-10-01T00-33-54-654/ANUFS_TSAL.kicad_pcb (KiCad board)
At the start: 2 copper layers, 30 parts, among them Q1 Q_NMOS_DGS, Q2 Q_NMOS_DGS, Q4 NPN, Q5 Q_NMOS_DGS, Q6 NPN, U1 ICM7555xB, U2 TLV172IDCK, U3 TLV172IDCK, U4 Optocoupler_DC_PhotoNPN_AKEC

Commit message: footprinted
Parts:
- moved U1 7.78 mm to (172.0, 91.9)
Changed lines of the file:
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@@
 	(footprint "Package_SO:SOIC-8_3.9x4.9mm_P1.27mm"
 		(layer "F.Cu")
-		(at 176.5 85.5)
+		(at 172.025 91.865)
 		(descr "SOIC, 8 Pin (JEDEC MS-012AA, https://www.analog.com/media/en/package-pcb-resources/package/pkg_pdf/soic_narrow-r/r_8.pdf)")
 		(tags "SOIC SO")
